File: YM2203_DeveloperBoard.kicad_sch (KiCad schematic)
At the start: 26 parts, among them J1 Conn_01x20_Pin, J2 Conn_01x20_Socket, J3 Conn_01x20_Socket, J4 Conn_01x20_Pin, J5 Conn_01x06_Socket, J6 AudioJack3, U3 MCP23S17_SP, U4 NJM4558, U5 NJM4558

Commit message: v2
Parts:
- added U6: ~, Package_TO_SOT_THT:TO-92_Inline_Wide, symbol OPN:Osc_TO92
Connections:
- net +5V: now also U6.3 (Vcc)
- net GND: now also U6.2 (GND)
- net OPN_ΦM: now also U6.1 (OUT)
Changed lines of the file:
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@@
+    (stroke (width 0) (type default))
+  )
+  (wire (pts (xy 224.79 43.18) (xy 227.33 43.18))
     (stroke (width 0) (type default))
   )
@@
     (stroke (width 0) (type default))
   )
+  (wire (pts (xy 224.79 45.72) (xy 224.79 46.99))
+    (stroke (width 0) (type default))
+  )
   (wire (pts (xy 162.56 59.69) (xy 177.8 59.69))
     (stroke (width 0) (type default))
@@
     (stroke (width 0) (type default))
   )
+  (wire (pts (xy 224.79 41.91) (xy 224.79 43.18))
+    (stroke (width 0) (type default))
+  )
   (wire (pts (xy 162.56 54.61) (xy 177.8 54.61))
     (stroke (width 0) (type default))
@@
     (stroke (width 0) (type default))
   )
+  (wire (pts (xy 227.33 45.72) (xy 224.79 45.72))
+    (stroke (width 0) (type default))
+  )
   (wire (pts (xy 193.04 92.71) (xy 201.93 92.71))
     (stroke (width 0) (type default))
@@
     (property "Intersheetrefs" "${INTERSHEET_REFS}" (at 100.7503 72.39 0)
       (effects (font (size 1.27 1.27)) (justify right) hide)
+    )
+  )
+  (global_label "OPN_ΦM" (shape output) (at 242.57 44.45 0) (fields_autoplaced)
+    (effects (font (size 1.27 1.27)) (justify left))
+    (property "Intersheetrefs" "${INTERSHEET_REFS}" (at 253.1563 44.45 0)
+      (effects (font (size 1.27 1.27)) (justify left) hide)
     )
   )
@@
         (path "/97dc443c-ac7e-46d6-a405-ba7928cfc411"
           (reference "#PWR023") (unit 1)
+        )
+      )
+    )
+  )
+  (symbol (lib_id "power:GND") (at 224.79 46.99 0) (unit 1)
+    (in_bom yes) (on_board yes) (dnp no) (fields_autoplaced)
+    (property "Reference" "#PWR025" (at 224.79 53.34 0)
+      (effects (font (size 1.27 1.27)) hide)
+    )
+    (property "Value" "GND" (at 224.79 52.07 0)
+      (effects (font (size 1.27 1.27)))
+    )
+    (property "Footprint" "" (at 224.79 46.99 0)
+      (effects (font (size 1.27 1.27)) hide)
+    )
+    (property "Datasheet" "" (at 224.79 46.99 0)
+      (effects (font (size 1.27 1.27)) hide)
+    )
+    (pin "1")
+    (instances
+      (project "YM2203_DeveloperBoard"
+        (path "/97dc443c-ac7e-46d6-a405-ba7928cfc411"
+          (reference "#PWR025") (unit 1)
         )
       )
@@
     )
   )
+  (symbol (lib_id "power:+5V") (at 224.79 41.91 0) (unit 1)
+    (in_bom yes) (on_board yes) (dnp no) (fields_autoplaced)
+    (property "Reference" "#PWR024" (at 224.79 45.72 0)
+      (effects (font (size 1.27 1.27)) hide)
+    )
+    (property "Value" "+5V" (at 224.79 38.1 0)
+      (effects (font (size 1.27 1.27)))
+    )
+    (property "Footprint" "" (at 224.79 41.91 0)
+      (effects (font (size 1.27 1.27)) hide)
+    )
+    (property "Datasheet" "" (at 224.79 41.91 0)
+      (effects (font (size 1.27 1.27)) hide)
+    )
+    (pin "1")
+    (instances
+      (project "YM2203_DeveloperBoard"
+        (path "/97dc443c-ac7e-46d6-a405-ba7928cfc411"
+          (reference "#PWR024") (unit 1)
+        )
+      )
+    )
+  )
   (symbol (lib_id "Device:R") (at 134.62 118.11 90) (unit 1)
     (in_bom yes) (on_board yes) (dnp no) (fields_autoplaced)
@@
         )
       )
+    )
+  )
+  (symbol (lib_id "OPN:Osc_TO92") (at 234.95 41.91 0) (unit 1)
+    (in_bom yes) (on_board yes) (dnp no) (fields_autoplaced)
+    (property "Reference" "U6" (at 234.95 40.64 0)
+      (effects (font (size 1.27 1.27)))
+    )
+    (property "Value" "~" (at 234.95 39.37 0)
+      (effects (font (size 1.27 1.27)))
+    )
+    (property "Footprint" "Package_TO_SOT_THT:TO-92_Inline_Wide" (at 234.95 39.37 0)
+      (effects (font (size 1.27 1.27)) hide)
+    )
+    (property "Datasheet" "" (at 234.95 39.37 0)
+      (effects (font (size 1.27 1.27)) hide)
+    )
+    (pin "1")
+    (pin "2")
+    (pin "3")
+    (instances
+      (project "YM2203_DeveloperBoard"
+        (path "/97dc443c-ac7e-46d6-a405-ba7928cfc411"
+          (reference "U6") (unit 1)
+        )
+      )
