File: YM2203_DeveloperBoard.kicad_pcb (KiCad board)
At the start: 2 copper layers, 99.1 x 99.1 mm, 27 parts, among them J1 Conn_01x20_Pin, J2 Conn_01x20_Socket, J3 Conn_01x20_Socket, J4 Conn_01x20_Pin, J5 Conn_01x06_Socket, J6 AudioJack3, U3 MCP23S17_SP, U4 NJM4558, U5 NJM4558

Commit message: update to v2
Parts:
- moved J5 5.08 mm to (218.4, 55.9)
Routing:
- net MCP_MISO: track 27.5 -> 25.4 mm
- net MCP_MOSI: track 30.0 -> 29.0 mm
- net MCP_#CS: track 35.1 -> 36.2 mm
Other:
- board text added: "1MHz OSC"
- board text removed: "1MHz"
Changed lines of the file:
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@@
   )
   (footprint "Connector_PinSocket_2.54mm:PinSocket_1x06_P2.54mm_Vertical" (layer "F.Cu")
-    (at 218.44 60.96)
+    (at 218.44 55.88)
     (descr "Through hole straight socket strip, 1x06, 2.54mm pitch, single row (from Kicad 4.0.7), script generated")
     (tags "Through hole socket strip THT 1x06 2.54mm single row")
@@
     (effects (font (size 1.5 1.5) (thickness 0.3) bold) (justify left))
   )
-  (gr_text "GND" (at 212.09 73.66) (layer "F.SilkS")
+  (gr_text "GND" (at 212.09 68.58) (layer "F.SilkS")
     (effects (font (size 1 1) (thickness 0.15)) (justify left))
   )
@@
     (effects (font (size 1.5 1.5) (thickness 0.3) bold) (justify left))
   )
-  (gr_text "+5V" (at 212.09 60.96) (layer "F.SilkS")
+  (gr_text "+5V" (at 212.09 55.88) (layer "F.SilkS")
     (effects (font (size 1 1) (thickness 0.15)) (justify left))
   )
@@
     (effects (font (size 1.5 1.5) (thickness 0.3) bold) (justify right))
   )
-  (gr_text "1MHz" (at 186.69 86.36) (layer "F.SilkS")
+  (gr_text "1MHz\nOSC" (at 186.69 86.36) (layer "F.SilkS")
     (effects (font (size 1.5 1.5) (thickness 0.2)) (justify top))
   )
@@
     (effects (font (size 1.5 1.5) (thickness 0.3) bold) (justify right))
   )
-  (gr_text "MCP23S17_MOSI" (at 203.2 68.915) (layer "F.SilkS")
+  (gr_text "MCP23S17_MOSI" (at 203.2 63.835) (layer "F.SilkS")
     (effects (font (size 1 1) (thickness 0.15)) (justify left))
   )
@@
     (effects (font (size 1.5 1.5) (thickness 0.3) bold) (justify right))
   )
-  (gr_text "MCP23S17_SCK" (at 203.2 66.375) (layer "F.SilkS")
+  (gr_text "MCP23S17_SCK" (at 203.2 61.295) (layer "F.SilkS")
     (effects (font (size 1 1) (thickness 0.15)) (justify left))
   )
@@
     (effects (font (size 1 1) (thickness 0.15)))
   )
-  (gr_text "MCP23S17_#CS" (at 203.2 63.835) (layer "F.SilkS")
+  (gr_text "MCP23S17_#CS" (at 203.2 58.755) (layer "F.SilkS")
     (effects (font (size 1 1) (thickness 0.15)) (justify left))
   )
-  (gr_text "MCP23S17_MISO" (at 203.2 71.455) (layer "F.SilkS")
+  (gr_text "MCP23S17_MISO" (at 203.2 66.375) (layer "F.SilkS")
     (effects (font (size 1 1) (thickness 0.15)) (justify left))
   )
@@
   (segment (start 187.96 124.46) (end 190.5 121.92) (width 0.25) (layer "B.Cu") (net 41))
   (segment (start 170.18 124.46) (end 187.96 124.46) (width 0.25) (layer "B.Cu") (net 41))
-  (segment (start 195.58 63.5) (end 194.31 62.23) (width 0.25) (layer "F.Cu") (net 42))
-  (segment (start 195.58 63.5) (end 218.44 63.5) (width 0.25) (layer "F.Cu") (net 42))
-  (segment (start 194.31 62.23) (end 189.23 62.23) (width 0.25) (layer "F.Cu") (net 42))
+  (segment (start 218.44 58.42) (end 214.63 62.23) (width 0.25) (layer "F.Cu") (net 42))
+  (segment (start 214.63 62.23) (end 189.23 62.23) (width 0.25) (layer "F.Cu") (net 42))
   (segment (start 189.23 62.23) (end 185.42 66.04) (width 0.25) (layer "F.Cu") (net 42))
+  (segment (start 218.44 60.96) (end 215.9 63.5) (width 0.25) (layer "F.Cu") (net 43))
   (segment (start 190.5 63.5) (end 187.96 66.04) (width 0.25) (layer "F.Cu") (net 43))
-  (segment (start 196.85 66.04) (end 194.31 63.5) (width 0.25) (layer "F.Cu") (net 43))
-  (segment (start 194.31 63.5) (end 190.5 63.5) (width 0.25) (layer "F.Cu") (net 43))
-  (segment (start 196.85 66.04) (end 218.44 66.04) (width 0.25) (layer "F.Cu") (net 43))
-  (segment (start 198.12 68.58) (end 218.44 68.58) (width 0.25) (layer "F.Cu") (net 44))
-  (segment (start 191.77 64.77) (end 194.31 64.77) (width 0.25) (layer "F.Cu") (net 44))
-  (segment (start 194.31 64.77) (end 198.12 68.58) (width 0.25) (layer "F.Cu") (net 44))
-  (segment (start 190.5 66.04) (end 191.77 64.77) (width 0.25) (layer "F.Cu") (net 44))
-  (segment (start 198.12 71.12) (end 218.44 71.12) (width 0.25) (layer "F.Cu") (net 45))
-  (segment (start 198.12 71.12) (end 193.04 66.04) (width 0.25) (layer "F.Cu") (net 45))
+  (segment (start 215.9 63.5) (end 190.5 63.5) (width 0.25) (layer "F.Cu") (net 43))
+  (segment (start 218.44 63.5) (end 217.17 64.77) (width 0.25) (layer "F.Cu") (net 44))
+  (segment (start 191.77 64.77) (end 190.5 66.04) (width 0.25) (layer "F.Cu") (net 44))
+  (segment (start 217.17 64.77) (end 191.77 64.77) (width 0.25) (layer "F.Cu") (net 44))
+  (segment (start 218.44 66.04) (end 193.04 66.04) (width 0.25) (layer "F.Cu") (net 45))
   (segment (start 185.42 58.42) (end 185.42 54.61) (width 0.25) (layer "F.Cu") (net 46))
   (segment (start 205.74 106.68) (end 205.73 106.69) (width 0.25) (layer "F.Cu") (net 47))
